Commit message: drive robot in sim

File: description/robot_core.xacro (robot description, xacro)
@@ -43,4 +43,9 @@
         </xacro:inertial_box>
     </link>
+    <gazebo reference="chassis">
+        <material>
+            Gazebo/White
+        </material>
+    </gazebo>
     <!-- LEFT WHEEL LINK -->
     <joint name="left_wheel_joint" type="continuous">
@@ -66,4 +71,9 @@
         </xacro:inertial_cylinder>
     </link>
+    <gazebo reference="left_wheel">
+        <material>
+            Gazebo/Blue
+        </material>
+    </gazebo>
     <!-- RIGHT WHEEL LINK -->
     <joint name="right_wheel_joint" type="continuous">
@@ -89,4 +99,9 @@
         </xacro:inertial_cylinder>
     </link>
+    <gazebo reference="right_wheel">
+        <material>
+            Gazebo/Blue
+        </material>
+    </gazebo>
     <!-- FRONT CASTER WHEEL LINK -->
     <joint name="front_caster_wheel_link" type="fixed">
@@ -111,4 +126,11 @@
         </xacro:inertial_sphere>
     </link>
+    <gazebo reference="front_caster_wheel">
+        <material>
+            Gazebo/Black
+        </material>
+        <mu1 value="0.001"/>
+        <mu2 value="0.001"/>
+    </gazebo>
     <!-- BACK CASTER WHEEL LINK -->
     <joint name="back_caster_wheel_link" type="fixed">
@@ -133,3 +155,8 @@
         </xacro:inertial_sphere>
     </link>
+    <gazebo reference="back_caster_wheel">
+        <material>Gazebo/Black</material>
+        <mu1 value="0.001"/>
+        <mu2 value="0.001"/>
+    </gazebo>
 </robot>

Commit message: Update left/right wheel

File: description/robot_core.xacro (robot description, xacro)
@@ -67,5 +67,6 @@
         <collision>
             <geometry>
-                <cylinder radius="0.07" length="0.04"/>
+                <sphere radius="0.07"/>
+                <!-- <cylinder radius="0.07" length="0.04"/> -->
             </geometry>
         </collision>
@@ -95,5 +96,6 @@
         <collision>
             <geometry>
-                <cylinder radius="0.07" length="0.04"/>
+                <sphere radius="0.07"/>
+                <!-- <cylinder radius="0.07" length="0.04"/> -->
             </geometry>
         </collision>
